Commit message: Add two rosbot in Gazebo/Rviz

File: src/rosbot_description/urdf/rosbot.xacro (robot description, xacro)
@@ -7,11 +7,11 @@
   <xacro:include filename="$(find rosbot_description)/urdf/materials.xacro" />
   <xacro:include filename="$(find rosbot_description)/urdf/rosbot.gazebo" />
-  <link name="base_link"></link>
+  <link name="$(arg robot_namespace)/base_link"></link>
   <joint name="base_link_joint" type="fixed">
     <origin xyz="0 0 0" rpy="0 0 0"/>
-    <parent link="base_link"/>
-    <child link="body_link"/>
-  </joint>
-  <link name='body_link'>
+    <parent link="$(arg robot_namespace)/base_link"/>
+    <child link="$(arg robot_namespace)/body_link"/>
+  </joint>
+  <link name='$(arg robot_namespace)/body_link'>
     <pose>0 0 0.1 0 0 0</pose>
     <inertial>
@@ -37,8 +37,8 @@
     <axis xyz="0 1 0" />
     <origin xyz="0 0 0" rpy="0 0 0"/>
-    <parent link="body_link"/>
-    <child link="top"/>
-  </joint>
-  <link name='top'>
+    <parent link="$(arg robot_namespace)/body_link"/>
+    <child link="$(arg robot_namespace)/top"/>
+  </joint>
+  <link name='$(arg robot_namespace)/top'>
     <pose>0 0 0 0 0 0</pose>
     <inertial>
@@ -55,5 +55,5 @@
     </visual>
   </link>
-  <link name="front_left_wheel">
+  <link name="$(arg robot_namespace)/front_left_wheel">
     <collision>
       <origin xyz="0 -0.014 0" rpy="${pi/2} 0 0"/>
@@ -83,5 +83,5 @@
     </inertial>
   </link>
-  <link name="front_right_wheel">
+  <link name="$(arg robot_namespace)/front_right_wheel">
     <collision>
       <origin xyz="0 0.014 0" rpy="${pi/2} 0 0"/>
@@ -111,5 +111,5 @@
     </inertial>
   </link>
-  <link name="rear_left_wheel">
+  <link name="$(arg robot_namespace)/rear_left_wheel">
     <collision>
       <origin xyz="0 -0.014 0" rpy="${pi/2} 0 0"/>
@@ -139,5 +139,5 @@
     </inertial>
   </link>
-  <link name="rear_right_wheel">
+  <link name="$(arg robot_namespace)/rear_right_wheel">
     <collision>
       <origin xyz="0 0.014 0" rpy="${pi/2} 0 0"/>
@@ -169,6 +169,6 @@
   <joint type="continuous" name="front_left_wheel_hinge">
     <origin xyz="0.05 0.11 0" rpy="0 0 0"/>
-    <child link="front_left_wheel"/>
-    <parent link="body_link"/>
+    <child link="$(arg robot_namespace)/front_left_wheel"/>
+    <parent link="$(arg robot_namespace)/body_link"/>
     <axis xyz="0 1 0" rpy="0 0 0"/>
     <limit effort="1" velocity="10"/>
@@ -186,6 +186,6 @@
   <joint type="continuous" name="front_right_wheel_hinge">
     <origin xyz="0.05 -0.11 0" rpy="0 0 0"/>
-    <child link="front_right_wheel"/>
-    <parent link="body_link"/>
+    <child link="$(arg robot_namespace)/front_right_wheel"/>
+    <parent link="$(arg robot_namespace)/body_link"/>
     <axis xyz="0 1 0" rpy="0 0 0"/>
     <limit effort="1" velocity="10"/>
@@ -203,6 +203,6 @@
   <joint type="continuous" name="rear_left_wheel_hinge">
     <origin xyz="-0.055 0.11 0" rpy="0 0 0"/>
-    <child link="rear_left_wheel"/>
-    <parent link="body_link"/>
+    <child link="$(arg robot_namespace)/rear_left_wheel"/>
+    <parent link="$(arg robot_namespace)/body_link"/>
     <axis xyz="0 1 0" rpy="0 0 0"/>
     <limit effort="1" velocity="10"/>
@@ -220,6 +220,6 @@
   <joint type="continuous" name="rear_right_wheel_hinge">
     <origin xyz="-0.055 -0.11 0" rpy="0 0 0"/>
-    <child link="rear_right_wheel"/>
-    <parent link="body_link"/>
+    <child link="$(arg robot_namespace)/rear_right_wheel"/>
+    <parent link="$(arg robot_namespace)/body_link"/>
     <axis xyz="0 1 0" rpy="0 0 0"/>
     <limit effort="1" velocity="10"/>
@@ -239,11 +239,11 @@
     <axis xyz="0 0 0" />
     <origin xyz="-0.03 0 0.18" rpy="0 0 0"/>
-    <parent link="body_link"/>
-    <child link="camera_link"/>
-  </joint>
-  <link name="camera_link">
+    <parent link="$(arg robot_namespace)/body_link"/>
+    <child link="$(arg robot_namespace)/camera_link"/>
+  </joint>
+  <link name="$(arg robot_namespace)/camera_link">
     <collision>
       <origin xyz="0.02 0 0" rpy="0 0 0"/>
-      <geometry>0
+      <geometry>
         <box size="0.001 0.001 0.001"/>
       </geometry>
@@ -264,24 +264,24 @@
   <joint name="camera_optical_joint" type="fixed">
     <origin xyz="0 0 0" rpy="${-pi/2} 0 ${-pi/2}"/>
-    <parent link="camera_link"/>
-    <child link="camera_rgb_frame"/>
-  </joint>
-  <link name="camera_rgb_frame">
+    <parent link="$(arg robot_namespace)/camera_link"/>
+    <child link="$(arg robot_namespace)/camera_rgb_frame"/>
+  </joint>
+  <link name="$(arg robot_namespace)/camera_rgb_frame">
   </link>
   <joint name="camera_depth_joint" type="fixed">
     <origin xyz="0 0 0" rpy="${-pi/2} 0 ${-pi/2}"/>
-    <parent link="camera_link"/>
-    <child link="camera_depth_frame"/>
-  </joint>
-  <link name="camera_depth_frame">
+    <parent link="$(arg robot_namespace)/camera_link"/>
+    <child link="$(arg robot_namespace)/camera_depth_frame"/>
+  </joint>
+  <link name="$(arg robot_namespace)/camera_depth_frame">
   </link>
   <joint name="rplidar_joint" type="fixed">
     <axis xyz="0 1 0" />
     <origin xyz="0.02 0 0.058" rpy="0 0 3.14"/>
-    <parent link="body_link"/>
-    <child link="laser"/>
+    <parent link="$(arg robot_namespace)/body_link"/>
+    <child link="$(arg robot_namespace)/laser"/>
   </joint>
   <!-- rplidar Laser -->
-  <link name="laser">
+  <link name="$(arg robot_namespace)/laser">
     <collision>
       <origin xyz="0 0 0" rpy="1.5707 0 4.71"/>
@@ -306,28 +306,28 @@
     <axis xyz="0 1 0" />
     <origin xyz="0.1 0.05 0.01" rpy="0 0 0.13 "/>
-    <parent link="body_link"/>
-    <child link="range_fl"/>
-  </joint>
-  <link name="range_fl"></link>
+    <parent link="$(arg robot_namespace)/body_link"/>
+    <child link="$(arg robot_namespace)/range_fl"/>
+  </joint>
+  <link name="$(arg robot_namespace)/range_fl"></link>
   <joint name="range_fr_joint" type="fixed">
     <axis xyz="0 1 0" />
     <origin xyz="0.1 -0.05 0.01" rpy="0 0 -0.13 "/>
-    <parent link="body_link"/>
-    <child link="range_fr"/>
-  </joint>
-  <link name="range_fr"></link>
+    <parent link="$(arg robot_namespace)/body_link"/>
+    <child link="$(arg robot_namespace)/range_fr"/>
+  </joint>
+  <link name="$(arg robot_namespace)/range_fr"></link>
   <joint name="range_rl_joint" type="fixed">
     <axis xyz="0 1 0" />
     <origin xyz="-0.1 0.05 0.01" rpy="0 0 3.01 "/>
-    <parent link="body_link"/>
-    <child link="range_rl"/>
-  </joint>
-  <link name="range_rl"></link>
+    <parent link="$(arg robot_namespace)/body_link"/>
+    <child link="$(arg robot_namespace)/range_rl"/>
+  </joint>
+  <link name="$(arg robot_namespace)/range_rl"></link>
   <joint name="range_rr_joint" type="fixed">
     <axis xyz="0 1 0" />
     <origin xyz="-0.1 -0.05 0.01" rpy="0 0 3.27 "/>
-    <parent link="body_link"/>
-    <child link="range_rr"/>
-  </joint>
-  <link name="range_rr"></link>
+    <parent link="$(arg robot_namespace)/body_link"/>
+    <child link="$(arg robot_namespace)/range_rr"/>
+  </joint>
+  <link name="$(arg robot_namespace)/range_rr"></link>
 </robot>

Commit message: Add TF map and odometry to the two robots

File: src/rosbot_description/urdf/rosbot.xacro (robot description, xacro)
@@ -3,4 +3,5 @@
   xmlns:xacro="http://www.ros.org/wiki/xacro">
   <xacro:arg name="robot_namespace" default=""/>
+  <!-- <xacro:arg name="init_y" default="0"/> -->
   <xacro:property name="cameraSize" value="0.05"/>
   <xacro:property name="cameraMass" value="0.1"/>
@@ -331,3 +332,29 @@
   </joint>
   <link name="$(arg robot_namespace)/range_rr"></link>
+  <!-- <gazebo>
+  <plugin name="ground_truth" filename="libgazebo_ros_p3d.so">
+    <frameName>world</frameName>
+    <bodyName>$(arg robot_namespace)/base_link</bodyName>
+    <topicName>$(arg robot_namespace)/odom</topicName>
+    <updateRate>30.0</updateRate>
+  </plugin>
+  </gazebo> -->
+ <!-- <link name="map">
+    <inertial>
+      <mass value="5"/>
+      <origin xyz="0 0 0.04" rpy=" 0 0 0"/>
+      <inertia ixx="0.01" ixy="0.01" ixz="0" iyy="0.01" iyz="0.01" izz="0.01" />
+    </inertial>
+  </link>
+ <joint name="map_joint" type="floating">
+    <parent link="map"/>
+    <child link="$(arg robot_namespace)/base_link"/>
+    <origin xyz="0 $(arg init_y) 0" rpy="0 0 0"/>
+ </joint>
+ <link name="top_link"/>
+ <joint name="top_joint" type="fixed">
+    <parent link="top_link"/>
+    <child link="map"/>
+    <origin xyz="0 0 0" rpy="0 0 0"/>
+ </joint> -->
 </robot>
